File: Group52HeatedBridgeKiCad - main/Group52HeatedBridge-2025-02-25_214848/Group52HeatedBridge.kicad_sch (KiCad schematic)
At the start: 32 parts, among them J1 UART, J10 TempSensorAirLED, J11 Regulator Vin, J12 54-00166, J2 RainSensor, J3 TemperatureSurface, J4 TemperatureAir, J5 JTAG, J6 TempSensorSurfaceLED, J7 RainSensor LED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

Commit message: power subsytem schematic - more chnages
Parts:
- added D2: 1N5820, Diode_THT:D_DO-201AD_P3.81mm_Vertical_KathodeUp, symbol Diode:1N5820
- added J13: Heater1, Connector_Molex:Molex_KK-254_AE-6410-02A_1x02_P2.54mm_Vertical, symbol Connector_Generic:Conn_01x02
- added J14: Heater2, Connector_Molex:Molex_KK-254_AE-6410-02A_1x02_P2.54mm_Vertical, symbol Connector_Generic:Conn_01x02
- added R10: 10, symbol Device:R
- added R11: 10k, symbol Device:R
Connections:
- net GND: now also U3.3 (S), R11.2
- net +24V: now reaches C4.1, C6.1, J12.1, U2.1 (VIN)
- net +24V: now also D2.1 (K), J13.1 (Pin_1), J14.1 (Pin_1)
- net at U3.1 (G): now also R10.2, R11.1
- net at U3.2 (D): now also D2.2 (A), J13.2 (Pin_2), J14.2 (Pin_2)
- new net MOSFETCONTROL: R10.1
Other:
- moved on the sheet: C4, C5, C6, D1, J12, L1, U2, U3

Commit message: power subsytem schematic push - second
Parts:
- removed J11: Regulator Vin, Connector_Molex:Molex_KK-254_AE-6410-02A_1x02_P2.54mm_Vertical, symbol Connector_Generic:Conn_01x02
- C4, C5, C6: footprint (none) -> Capacitor_SMD:C_0805_2012Metric_Pad1.18x1.45mm_HandSolder
- J12: footprint CONN3_54-00166_TEN -> footprints_barrel:CONN3_54-00166_TEN
- L1: footprint (none) -> Inductor_SMD:L_0805_2012Metric_Pad1.15x1.40mm_HandSolder
- R10, R11: footprint (none) -> Resistor_SMD:R_0805_2012Metric_Pad1.20x1.40mm_HandSolder
- U3: footprint PG-TO220-3_INF -> footprints:PG-TO220-3_INF
Connections:
- net +3.3V: now also U2.3 (FB)
- net MOSFETCONTROL: now also U1.11 (IO26)
