File: Group52HeatedBridgeKiCad - main/Group52HeatedBridge-2025-02-25_214848/Group52HeatedBridge.kicad_sch (KiCad schematic)
At the start: 36 parts, among them J1 UART, J10 TempSensorAirLED, J12 54-00166, J13 Heater1, J14 Heater2, J2 RainSensor, J3 TemperatureSurface, J4 TemperatureAir, J5 JTAG, J6 TempSensorSurfaceLED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

Commit message: B Revert "resized schematic and cleaned up"
This reverts commit bab35e5b8986f5439bb45f55d315508e4487ff8d.

reverted auto save file
Changed lines of the file:
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@@
 (kicad_sch
-	(version 20250114)
+	(version 20231120)
 	(generator "eeschema")
-	(generator_version "9.0")
+	(generator_version "8.0")
 	(paper "A1")
 	(junction
@@
 	(label "MTCK"
 		(at 485.14 116.84 0)
+		(fields_autoplaced yes)
 		(effects
 			(font
@@
 	(label "BOOT"
 		(at 375.92 119.38 0)
+		(fields_autoplaced yes)
 		(effects
 			(font
@@
 	(label "GPIOTempSurfaceLED"
 		(at 375.92 144.78 0)
+		(fields_autoplaced yes)
 		(effects
 			(font
@@
 	(label "EN"
 		(at 336.55 119.38 0)
+		(fields_autoplaced yes)
 		(effects
 			(font
@@
 	(label "MTDI"
 		(at 485.14 119.38 0)
+		(fields_autoplaced yes)
 		(effects
 			(font
@@
 	(label "MOSFETCONTROL"
 		(at 182.88 38.1 0)
+		(fields_autoplaced yes)
 		(effects
 			(font
@@
 	(label "MTMS"
 		(at 485.14 121.92 0)
+		(fields_autoplaced yes)
 		(effects
 			(font
@@
 	(label "GPIORainLED"
 		(at 374.65 172.72 0)
+		(fields_autoplaced yes)
 		(effects
 			(font
@@
 	(label "AnalogRain"
 		(at 374.65 177.8 0)
+		(fields_autoplaced yes)
 		(effects
 			(font
@@
 	(label "GPIOTempAirLED"
 		(at 375.92 149.86 0)
+		(fields_autoplaced yes)
 		(effects
 			(font
@@
 	(label "MTDO"
 		(at 375.92 142.24 0)
+		(fields_autoplaced yes)
 		(effects
 			(font
@@
 	(label "DigitalRain"
 		(at 374.65 175.26 0)
+		(fields_autoplaced yes)
 		(effects
 			(font
@@
 	(label "MTMS"
 		(at 375.92 139.7 0)
+		(fields_autoplaced yes)
 		(effects
 			(font
@@
 	(label "RX"
 		(at 375.92 127 0)
+		(fields_autoplaced yes)
 		(effects
 			(font
@@
 	(label "MOSFETCONTROL"
 		(at 373.38 165.1 0)
+		(fields_autoplaced yes)
 		(effects
 			(font
@@
 	(label "GPIOTempSurface"
 		(at 375.92 147.32 0)
+		(fields_autoplaced yes)
 		(effects
 			(font
@@
 	(label "MTDO"
 		(at 485.14 114.3 0)
+		(fields_autoplaced yes)
 		(effects
 			(font
@@
 	(label "GPIOTempAir"
 		(at 375.92 152.4 0)
+		(fields_autoplaced yes)
 		(effects
 			(font
@@
 	(label "MTCK"
 		(at 375.92 137.16 0)
+		(fields_autoplaced yes)
 		(effects
 			(font
@@
 	(label "MTDI"
 		(at 375.92 134.62 0)
+		(fields_autoplaced yes)
 		(effects
 			(font
@@
 	(label "TX"
 		(at 375.92 121.92 0)
+		(fields_autoplaced yes)
 		(effects
 			(font
@@
 		)
 	)
-	(embedded_fonts no)
 )
