File: Group52HeatedBridge-resized/Group52HeatedBridge.kicad_pcb (KiCad board)
At the start: 2 copper layers, 100 x 100 mm, 24 parts, among them J1 UART, J10 TempSensorAirLED, J2 RainSensor, J3 TemperatureSurface, J4 TemperatureAir, J5 JTAG, J6 TempSensorSurfaceLED, J7 RainSensor LED, J8 EN_BUTTON, J9 BOOT_BUTTON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

Commit message: passes pcbway audit
Parts:
- added C4: 470uf, Capacitor_SMD:C_0805_2012Metric_Pad1.18x1.45mm_HandSolder, F.Cu at (130.9, 121.8)
- added C5: 330uf, Capacitor_SMD:C_0805_2012Metric_Pad1.18x1.45mm_HandSolder, F.Cu at (117.0, 113.0)
- added C6: 1uf, Capacitor_SMD:C_0805_2012Metric_Pad1.18x1.45mm_HandSolder, F.Cu at (130.8, 117.7)
- added D1: 1N5820, Diode_THT:D_DO-201AD_P3.81mm_Vertical_KathodeUp, F.Cu at (106.8, 108.6)
- added D2: 1N5820, Diode_THT:D_DO-201AD_P3.81mm_Vertical_KathodeUp, F.Cu at (145.7, 126.6)
- added J11: 54-00166, 54_00166_2:TENSILITY_54-00166, F.Cu at (129.4, 131.6)
- added J13: Heater1, Connector_Molex:Molex_KK-254_AE-6410-02A_1x02_P2.54mm_Vertical, F.Cu at (154.6, 122.7)
- added J14: Heater2, Connector_Molex:Molex_KK-254_AE-6410-02A_1x02_P2.54mm_Vertical, F.Cu at (152.5, 112.4)
- added L1: 47uh, Inductor_SMD:L_0805_2012Metric_Pad1.15x1.40mm_HandSolder, F.Cu at (108.6, 114.9)
- added R10: 10, Resistor_SMD:R_0805_2012Metric_Pad1.20x1.40mm_HandSolder, F.Cu at (142.6, 137.2)
- added R11: 10k, Resistor_SMD:R_0805_2012Metric_Pad1.20x1.40mm_HandSolder, F.Cu at (143.6, 132.5)
- added U3: IRLZ44NPBF, footprints_mosfet:PG-TO220-3_INF, F.Cu at (154.1, 133.9)
- moved U2 0.45 mm to (113.4, 125.1)
Routing:
- net GND: track 229.4 -> 321.0 mm, vias 5 -> 11
- net /MOSFETCONTROL: track 0.00 -> 69.3 mm, vias 0 -> 2
- net +24V: track 0.00 -> 68.7 mm
- net Net-(D2-A): track 0.00 -> 58.7 mm
- net +3.3V: track 362.6 -> 395.9 mm
- net Net-(D1-K): track 0.00 -> 17.8 mm
- net Net-(U3-G): track 0.00 -> 16.9 mm
Other:
- board text added: "Heated Bridge V1 03-03-2025 Group 52"
