File: Group52HeatedBridge-resized/Group52HeatedBridge.kicad_sch (KiCad schematic)
At the start: 36 parts, among them J1 UART, J10 TempSensorAirLED, J12 54-00166, J13 Heater1, J14 Heater2, J2 RainSensor, J3 TemperatureSurface, J4 TemperatureAir, J5 JTAG, J6 TempSensorSurfaceLED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

Commit message: passes pcbway audit
Parts:
- added J11: 54-00166, 54_00166_2:TENSILITY_54-00166, symbol 54-00166:54-00166
- J12: footprint footprints_barrel:CONN3_54-00166_TEN -> 54_00166_2:TENSILITY_54-00166
- U3: footprint footprints:PG-TO220-3_INF -> footprints_mosfet:PG-TO220-3_INF
Connections:
- net +24V: now also J11.A; no longer J12.1
- net GND: now also J11.B; no longer J12.3
Other:
- moved on the sheet: J12
Changed lines of the file:
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@@
 	)
 	(no_connect
-		(at 210.82 72.39)
-	)
-	(no_connect
 		(at 342.9 124.46)
 	)
@@
 	)
 	(no_connect
+		(at 204.47 72.39)
+	)
+	(no_connect
 		(at 373.38 132.08)
 	)
@@
 	(wire
 		(pts
+			(xy 207.01 69.85) (xy 204.47 69.85)
+		)
+		(stroke
+			(width 0)
+			(type default)
+		)
+	)
+	(wire
+		(pts
 			(xy 317.5 111.76) (xy 314.96 111.76)
 		)
@@
 	(wire
 		(pts
+			(xy 204.47 74.93) (xy 210.82 74.93)
+		)
+		(stroke
+			(width 0)
+			(type default)
+		)
+	)
+	(wire
+		(pts
 			(xy 278.13 27.94) (xy 278.13 22.86)
 		)
@@
 	(wire
 		(pts
+			(xy 207.01 67.31) (xy 228.6 67.31)
+		)
+		(stroke
+			(width 0)
+			(type default)
+		)
+	)
+	(wire
+		(pts
 			(xy 406.4 87.63) (xy 406.4 90.805)
 		)
@@
 	(wire
 		(pts
+			(xy 210.82 77.47) (xy 210.82 74.93)
+		)
+		(stroke
+			(width 0)
+			(type default)
+		)
+	)
+	(wire
+		(pts
 			(xy 434.975 107.315) (xy 434.975 142.24)
 		)
@@
 	(wire
 		(pts
-			(xy 210.82 67.31) (xy 228.6 67.31)
-		)
-		(stroke
-			(width 0)
-			(type default)
-		)
-	)
-	(wire
-		(pts
 			(xy 302.26 53.34) (xy 302.26 59.69)
 		)
@@
 	(wire
 		(pts
+			(xy 207.01 67.31) (xy 207.01 69.85)
+		)
+		(stroke
+			(width 0)
+			(type default)
+		)
+	)
+	(wire
+		(pts
 			(xy 425.45 160.02) (xy 425.45 162.56)
 		)
@@
 	(symbol
 		(lib_id "2025-02-28_21-13-51:54-00166")
-		(at 210.82 67.31 0)
+		(at 133.35 54.61 0)
 		(unit 1)
 		(exclude_from_sim no)
@@
 		(fields_autoplaced yes)
 		(property "Reference" "J12"
-			(at 198.12 59.69 0)
+			(at 120.65 46.99 0)
 			(effects
 				(font
@@
 		)
 		(property "Value" "54-00166"
-			(at 198.12 62.23 0)
+			(at 120.65 49.53 0)
 			(effects
 				(font
@@
 			)
 		)
-		(property "Footprint" "footprints_barrel:CONN3_54-00166_TEN"
-			(at 210.82 67.31 0)
+		(property "Footprint" "54_00166_2:TENSILITY_54-00166"
+			(at 133.35 54.61 0)
 			(effects
 				(font
@@
 		)
 		(property "Datasheet" "54-00166"
-			(at 210.82 67.31 0)
+			(at 133.35 54.61 0)
 			(effects
 				(font
@@
 		)
 		(property "Description" ""
-			(at 210.82 67.31 0)
+			(at 133.35 54.61 0)
 			(effects
 				(font
@@
 		)
 		(instances
-			(project ""
+			(project "Group52HeatedBridge"
 				(path "/bb48adda-4915-4436-95dc-e9dcb2cba51b"
 					(reference "J12")
@@
 			)
 		)
-		(property "Footprint" "footprints:PG-TO220-3_INF"
+		(property "Footprint" "footprints_mosfet:PG-TO220-3_INF"
 			(at 233.68 38.1 0)
 			(effects
@@
 					(unit 1)
 				)
+			)
+		)
+	)
+	(symbol
+		(lib_id "54-00166:54-00166")
+		(at 199.39 72.39 0)
+		(unit 1)
+		(exclude_from_sim no)
+		(in_bom yes)
+		(on_board yes)
+		(dnp no)
+		(fields_autoplaced yes)
+		(property "Reference" "J11"
+			(at 194.6303 63.5 0)
+			(effects
+				(font
+					(size 1.27 1.27)
+				)
+			)
+		)
+		(property "Value" "54-00166"
+			(at 194.6303 66.04 0)
+			(effects
+				(font
+					(size 1.27 1.27)
+				)
+			)
+		)
+		(property "Footprint" "54_00166_2:TENSILITY_54-00166"
+			(at 199.39 72.39 0)
+			(effects
+				(font
+					(size 1.27 1.27)
+				)
+				(justify bottom)
+				(hide yes)
+			)
+		)
+		(property "Datasheet" ""
+			(at 199.39 72.39 0)
+			(effects
+				(font
+					(size 1.27 1.27)
+				)
+				(hide yes)
+			)
+		)
+		(property "Description" ""
+			(at 199.39 72.39 0)
+			(effects
+				(font
+					(size 1.27 1.27)
+				)
+				(hide yes)
+			)
+		)
+		(property "PARTREV" "A"
+			(at 199.39 72.39 0)
+			(effects
+				(font
+					(size 1.27 1.27)
+				)
+				(justify bottom)
+				(hide yes)
+			)
+		)
+		(property "STANDARD" "Manufacturer Recommendations"
+			(at 199.39 72.39 0)
+			(effects
+				(font
+					(size 1.27 1.27)
+				)
+				(justify bottom)
+				(hide yes)
+			)
+		)
+		(property "SNAPEDA_PN" "54-00166"
+			(at 199.39 72.39 0)
+			(effects
+				(font
+					(size 1.27 1.27)
+				)
+				(justify bottom)
+				(hide yes)
+			)
+		)
+		(property "MAXIMUM_PACKAGE_HEIGHT" "11.2mm"
+			(at 199.39 72.39 0)
+			(effects
+				(font
+					(size 1.27 1.27)
+				)
+				(justify bottom)
+				(hide yes)
+			)
+		)
+		(property "MANUFACTURER" "TENSILITY"
+			(at 199.39 72.39 0)
+			(effects
+				(font
+					(size 1.27 1.27)
+				)
+				(justify bottom)
+				(hide yes)
+			)
+		)
+		(pin "C"
+		)
+		(pin "B"
+		)
+		(pin "A"
+		)
+		(instances
+			(project ""
+				(path "/bb48adda-4915-4436-95dc-e9dcb2cba51b"
+					(reference "J11")
+					(unit 1)
+				)
